File: controllerBoard/board.kicad_pcb (KiCad board)
At the start: 2 copper layers, 100 x 50 mm, 12 parts, among them J1 Screw_Terminal_01x10, U1 TBD62783A, U2 TBD62783A

Commit message: Improve pcb +  error handling in firmware
Parts:
- added C1: 100nF, Capacitor_SMD:C_0805_2012Metric_Pad1.18x1.45mm_HandSolder, F.Cu at (136.0, 115.0)
- added C2: 100nF, Capacitor_SMD:C_0805_2012Metric_Pad1.18x1.45mm_HandSolder, F.Cu at (206.0, 121.0)
- added C3: 25v/100uF, Capacitor_THT:CP_Radial_Tantal_D6.0mm_P5.00mm, F.Cu at (204.5, 133.0)
- added D1: LED, LED_SMD:LED_0805_2012Metric_Pad1.15x1.40mm_HandSolder, F.Cu at (124.9, 136.5)
- added J2: Barrel_Jack, Connector_BarrelJack:BarrelJack_CUI_PJ-079BH_Horizontal, F.Cu at (212.4, 143.6)
- added R19: 330, Resistor_SMD:R_1206_3216Metric, F.Cu at (131.0, 136.5)
- added U3: ESP32-WROOM-32U, PCM_Espressif:ESP32-DevKitC, F.Cu at (187.9, 111.3)
- R10, R11, R12, R13, R14, R15, R16, R17, R18: value 110 -> 82
- U1, U2: value TBD62783A -> TD62783AD
- moved U2 15.3 mm to (201.9, 111.8)
- moved U1 14.8 mm to (125.7, 115.0)
- moved R10 11.5 mm to (120.0, 102.0), turned to 180 degrees
- moved R14 11.0 mm to (158.8, 102.0), turned to 180 degrees
- moved R15 8.77 mm to (170.0, 102.0)
- moved R11 6.29 mm to (129.2, 102.0), turned to 180 degrees
- moved R18 6.28 mm to (200.0, 102.0)
- moved R13 5.07 mm to (148.8, 102.0), turned to 180 degrees
- moved R16 3.80 mm to (180.0, 102.0)
- moved R17 1.39 mm to (190.0, 102.0)
- moved R12 1.17 mm to (138.6, 102.0), turned to 180 degrees
Connections:
- U1 pad 1: unconnected-(U1-I1-Pad1) -> Net-(U1-I1)
- U1 pad 2: unconnected-(U1-I2-Pad2) -> Net-(U1-I2)
- U1 pad 3: unconnected-(U1-I3-Pad3) -> Net-(U1-I3)
- U1 pad 4: unconnected-(U1-I4-Pad4) -> Net-(U1-I4)
- U1 pad 5: unconnected-(U1-I5-Pad5) -> Net-(U1-I5)
- U1 pad 6: unconnected-(U1-I6-Pad6) -> GND
- U1 pad 7: unconnected-(U1-I7-Pad7) -> GND
- U1 pad 8: unconnected-(U1-I8-Pad8) -> GND
- U2 pad 1: unconnected-(U2-I1-Pad1) -> Net-(U2-I1)
- U2 pad 2: unconnected-(U2-I2-Pad2) -> Net-(U2-I2)
- U2 pad 3: unconnected-(U2-I3-Pad3) -> Net-(U2-I3)
- U2 pad 4: unconnected-(U2-I4-Pad4) -> Net-(U2-I4)
- U2 pad 5: unconnected-(U2-I5-Pad5) -> GND
- U2 pad 6: unconnected-(U2-I6-Pad6) -> GND
- U2 pad 7: unconnected-(U2-I7-Pad7) -> GND
- U2 pad 8: unconnected-(U2-I8-Pad8) -> GND
Routing:
- net GND: track 0.00 -> 44.0 mm, vias 0 -> 2
- net Net-(U1-O5): track 0.00 -> 35.6 mm, vias 0 -> 2
- net Net-(U1-O4): track 0.00 -> 32.6 mm, vias 0 -> 2
- net Net-(U1-O3): track 0.00 -> 18.8 mm
- net Net-(J1-Pin_1): track 0.00 -> 17.1 mm
- net Net-(J1-Pin_2): track 0.00 -> 15.5 mm
- net Net-(J1-Pin_3): track 0.00 -> 15.4 mm
- net Net-(J1-Pin_4): track 0.00 -> 15.4 mm
- net +12V: track 0.00 -> 12.4 mm
- net Net-(U1-O2): track 0.00 -> 11.8 mm
- net Net-(J1-Pin_9): track 0.00 -> 11.6 mm
- net Net-(J1-Pin_8): track 0.00 -> 11.6 mm
- net Net-(J1-Pin_7): track 0.00 -> 11.6 mm
- net Net-(J1-Pin_6): track 0.00 -> 11.6 mm
- net Net-(U1-O1): track 0.00 -> 11.2 mm
Other:
- board size 100 x 50 mm -> 100 x 75 mm
