File: controllerBoard/board.kicad_sch (KiCad schematic)
At the start: 12 parts, among them J1 Screw_Terminal_01x10, U1 TBD62783A, U2 TBD62783A

Commit message: Improve pcb +  error handling in firmware
Parts:
- added C1, C2: 100nF, Capacitor_SMD:C_0805_2012Metric_Pad1.18x1.45mm_HandSolder, symbol Device:C
- added C3: 25v/100uF, Capacitor_THT:CP_Radial_Tantal_D6.0mm_P5.00mm, symbol Device:C_Polarized
- added D1: LED, LED_SMD:LED_0805_2012Metric_Pad1.15x1.40mm_HandSolder, symbol Device:LED
- added J2: Barrel_Jack, Connector_BarrelJack:BarrelJack_CUI_PJ-079BH_Horizontal, symbol Connector:Barrel_Jack
- added R19: 330, Resistor_SMD:R_1206_3216Metric, symbol Device:R_Small
- added U3: ESP32-WROOM-32U, PCM_Espressif:ESP32-DevKitC, symbol RF_Module:ESP32-WROOM-32U
- R10, R11, R12, R13, R14, R15, R16, R17, R18: value 110 -> 82
- U1, U2: value TBD62783A -> TD62783AD
Connections:
- net +12V: now also C1.2, C2.2, C3.1, J2.1
- net GND: now also U1.6 (I6), U1.7 (I7), U1.8 (I8), U2.5 (I5), U2.6 (I6), U2.7 (I7), U2.8 (I8), C1.1, C2.1, C3.2, D1.1 (K), J2.2, U3.1 (GND), U3.15 (GND), U3.38 (GND), U3.39 (GND)
- net at U2.1 (I1): now also U3.11 (IO26)
- net at U2.2 (I2): now also U3.12 (IO27)
- net at U2.3 (I3): now also U3.8 (IO32)
- net at U2.4 (I4): now also U3.9 (IO33)
- net at U1.1 (I1): now also U3.30 (IO18)
- net at U1.2 (I2): now also U3.33 (IO21)
- net at U1.3 (I3): now also U3.36 (IO22)
- net at U1.4 (I4): now also U3.37 (IO23)
- net at U1.5 (I5): now also U3.10 (IO25)
- new net: D1.2 (A), R19.1
- new net: R19.2, U3.31 (IO19)
- new net +5V: U3.2 (VDD)
- no-connect marks 0 -> 7
